Commit message: final changes

File: own_ur_description_2/urdf/ur_macro.xacro (robot description, xacro)
@@ -446,5 +446,5 @@
     </joint>
     <joint name="camera_joint" type="fixed">
-<origin xyz="0.0 0.06 0.045" rpy="1.5707 -1.5707 0.0"/>
+<origin xyz="0.0 0.065 0.05" rpy="1.5707 -1.5707 0.0"/>
         <parent link="wrist_3_link"/>
         <child link="camera_link"/>
